Commit message: ready to make the experiments of drawing

File: urdf/panda_calibrated_left.urdf (robot description, URDF)
Before this commit: robot panda, 14 links, 13 joints
Joints:
- joint ball_joint: origin xyz=0.00037990524928465026 -4.420572608777121e-05 0.03102464075322382 rpy=0.0 0.0 0.0 -> xyz=-8.138033409441562e-05 -5.6435696017550334e-05 0.03135847277442007 rpy=0.0 0.0 0.0
- joint panda_joint1: origin xyz=-1.2758753865242616e-16 -5.2222054042510136e-17 0.333 rpy=8.366805516041043e-06 8.814350308898128e-08 2.4513630387076608e-17 -> xyz=2.165725341166756e-17 -8.5102190577066e-17 0.333 rpy=-7.951740496840122e-18 -1.6002016950875694e-17 -6.409999329822744e-17
- joint panda_joint2: origin xyz=-0.00019417564815309772 -0.00018772077543271004 1.796911857934499e-17 rpy=-1.5725347107345484 0.0009255042963167639 -2.2321032908662564e-15 -> xyz=2.7011907872371278e-05 -0.0002976433617619205 -2.301983990164113e-18 rpy=-1.5726718418128585 0.0008795362448001076 -1.1830133872921954e-08
- joint panda_joint3: origin xyz=0.0003371033096498455 -0.31626505724737547 -0.0001877201793910496 rpy=1.5720487481374692 0.00011271550591184526 0.0008189810488676046 -> xyz=0.0002587677690204907 -0.31592427862323635 -0.00029763832100456757 rpy=1.5724513592285052 0.0009517599873760647 0.000797582477804661
- joint panda_joint4: origin xyz=0.08250428687456778 -0.0002847200612681194 0.0002655680887159182 rpy=1.5741434757926136 0.011776708120902118 -9.025189862699405e-05 -> xyz=0.08195228403580808 0.00014828533797593539 -7.510120361854353e-05 rpy=1.5725876195118216 0.011395465980731502 -0.0009652872714631131
- joint panda_joint5: origin xyz=-0.07866941844576122 0.38493907517903264 0.000283829074942361 rpy=-1.569359416779495 0.005129171736623614 -0.01022805489571219 -> xyz=-0.07854177795180825 0.3846146261676666 -0.00014727977826979903 rpy=-1.5714223242470033 0.004883367342631799 -0.009822564315057248
- joint panda_joint6: origin xyz=0.0006537446895798644 -1.275492785867517e-05 0.0009786397273711831 rpy=1.5705258868617893 -0.00043533480446275005 0.005114480048959338 -> xyz=0.0006322258545794781 0.00020292864991245296 0.0006540051425123762 rpy=1.5719531158024398 -0.0005298833733962498 0.004889463662293645
- joint panda_joint7: origin xyz=0.0902493646325364 -0.0008951821978016663 1.636289653042385e-05 rpy=1.5707208785930096 2.6320186308338895e-08 0.0005154940135814471 -> xyz=0.09012577560395825 2.5216340689147795e-06 -0.0002005371742828918 rpy=1.5708418247986804 -1.0867383571883744e-08 0.0005239043043533068

File: urdf/panda_calibrated_right.urdf (robot description, URDF)
Before this commit: robot panda, 14 links, 13 joints
Joints:
- joint ball_joint: origin xyz=0.00037990524928465026 -4.420572608777121e-05 0.03102464075322382 rpy=0.0 0.0 0.0 -> xyz=-0.0002660872941297353 -0.0006013031151721279 0.03213867409590657 rpy=0.0 0.0 0.0
- joint panda_joint1: origin xyz=-1.2758753865242616e-16 -5.2222054042510136e-17 0.333 rpy=8.366805516041043e-06 8.814350308898128e-08 2.4513630387076608e-17 -> xyz=3.92306549994108e-17 -1.8882042510814725e-17 0.333 rpy=-4.149806467317431e-18 7.137365686697144e-18 -4.589661264154907e-17
- joint panda_joint2: origin xyz=-0.00019417564815309772 -0.00018772077543271004 1.796911857934499e-17 rpy=-1.5725347107345484 0.0009255042963167639 -2.2321032908662564e-15 -> xyz=0.00019948308971021362 8.224025617840919e-05 -4.520794936045981e-18 rpy=-1.569171687032732 0.00044804054045514627 3.716085806330908e-08
- joint panda_joint3: origin xyz=0.0003371033096498455 -0.31626505724737547 -0.0001877201793910496 rpy=1.5720487481374692 0.00011271550591184526 0.0008189810488676046 -> xyz=-4.831237243079438e-05 -0.3160196186961809 8.223830388911502e-05 rpy=1.5701368639143456 0.00021547124952556483 0.00046325645207522415
- joint panda_joint4: origin xyz=0.08250428687456778 -0.0002847200612681194 0.0002655680887159182 rpy=1.5741434757926136 0.011776708120902118 -9.025189862699405e-05 -> xyz=0.08218622382442696 0.00012463089813243814 1.9815805120017282e-05 rpy=1.5699691608784458 0.003392401284735163 -0.00022561343078897857
- joint panda_joint5: origin xyz=-0.07866941844576122 0.38493907517903264 0.000283829074942361 rpy=-1.569359416779495 0.005129171736623614 -0.01022805489571219 -> xyz=-0.08161671980459631 0.38418467132228995 -0.0001250123513799326 rpy=-1.5712115657202819 0.0016558929683474796 -0.0030382657944411353
- joint panda_joint6: origin xyz=0.0006537446895798644 -1.275492785867517e-05 0.0009786397273711831 rpy=1.5705258868617893 -0.00043533480446275005 0.005114480048959338 -> xyz=6.629314849055931e-05 0.00045553055999363366 0.00018813569080110683 rpy=1.5680134729931703 8.562990901120595e-05 0.0016569948945247314
- joint panda_joint7: origin xyz=0.0902493646325364 -0.0008951821978016663 1.636289653042385e-05 rpy=1.5707208785930096 2.6320186308338895e-08 0.0005154940135814471 -> xyz=0.08768107566644284 -1.2646922078415426e-05 -0.0004545969030486451 rpy=1.5708928447112276 -1.1846509241174548e-07 -7.997671792020968e-05

Commit message: added the new calibrated models

File: urdf/panda_calibrated_left.urdf (robot description, URDF)
Before this commit: robot panda, 14 links, 13 joints
Joints:
- joint ball_joint: origin xyz=-8.138033409441562e-05 -5.6435696017550334e-05 0.03135847277442007 rpy=0.0 0.0 0.0 -> xyz=-0.00023049759980861887 0.00044039014121866966 0.031100743489190348 rpy=0.0 0.0 0.0
- joint panda_joint1: origin xyz=2.165725341166756e-17 -8.5102190577066e-17 0.333 rpy=-7.951740496840122e-18 -1.6002016950875694e-17 -6.409999329822744e-17 -> xyz=-1.4596613238343867e-17 -9.055693218673766e-17 0.333 rpy=-1.828892248693048e-17 8.671137250584476e-18 -2.0577862275452234e-17
- joint panda_joint2: origin xyz=2.7011907872371278e-05 -0.0002976433617619205 -2.301983990164113e-18 rpy=-1.5726718418128585 0.0008795362448001076 -1.1830133872921954e-08 -> xyz=0.00034046892346445374 -0.00027609138626588024 -2.4530901909373608e-17 rpy=-1.5731826118735361 0.0008804625507391334 4.79318753789608e-08
- joint panda_joint3: origin xyz=0.0002587677690204907 -0.31592427862323635 -0.00029763832100456757 rpy=1.5724513592285052 0.0009517599873760647 0.000797582477804661 -> xyz=0.00011482204889668299 -0.31591360277075664 -0.0002760912953803214 rpy=1.5723422152643884 0.0008208410846264723 0.0008441267498452069
- joint panda_joint4: origin xyz=0.08195228403580808 0.00014828533797593539 -7.510120361854353e-05 rpy=1.5725876195118216 0.011395465980731502 -0.0009652872714631131 -> xyz=0.08225834378378427 -2.2463482153615717e-05 -8.565172079819686e-05 rpy=1.5731556140861436 0.011786197996681824 -0.0008202845766085335
- joint panda_joint5: origin xyz=-0.07854177795180825 0.3846146261676666 -0.00014727977826979903 rpy=-1.5714223242470033 0.004883367342631799 -0.009822564315057248 -> xyz=-0.07855928728215028 0.38451520959214897 2.294719504146994e-05 rpy=-1.5706656685042597 0.004904763353391575 -0.010228702256771381
- joint panda_joint6: origin xyz=0.0006322258545794781 0.00020292864991245296 0.0006540051425123762 rpy=1.5719531158024398 -0.0005298833733962498 0.004889463662293645 -> xyz=0.0006528784687554265 0.00019996069776008653 0.0005556285825519909 rpy=1.5717644448432413 -0.0005146035481431135 0.0049033457862993225
- joint panda_joint7: origin xyz=0.09012577560395825 2.5216340689147795e-06 -0.0002005371742828918 rpy=1.5708418247986804 -1.0867383571883744e-08 0.0005239043043533068 -> xyz=0.09024626292728476 -2.4012052499956137e-05 -0.0001973603029375395 rpy=1.5708497729215354 -5.006328509410342e-08 0.0005117785060925037

File: urdf/panda_calibrated_right.urdf (robot description, URDF)
Before this commit: robot panda, 14 links, 13 joints
Joints:
- joint ball_joint: origin xyz=-0.0002660872941297353 -0.0006013031151721279 0.03213867409590657 rpy=0.0 0.0 0.0 -> xyz=0.0002309827402522288 -0.0004328828032887883 0.03240671849867958 rpy=0.0 0.0 0.0
- joint panda_joint1: origin xyz=3.92306549994108e-17 -1.8882042510814725e-17 0.333 rpy=-4.149806467317431e-18 7.137365686697144e-18 -4.589661264154907e-17 -> xyz=-6.283931712402919e-18 5.785240799539949e-17 0.333 rpy=2.4213079838489953e-17 -3.589660391516474e-18 -8.469944304901584e-18
- joint panda_joint2: origin xyz=0.00019948308971021362 8.224025617840919e-05 -4.520794936045981e-18 rpy=-1.569171687032732 0.00044804054045514627 3.716085806330908e-08 -> xyz=-0.00010087933252105225 0.0001070930255027192 1.7329529520611466e-17 rpy=-1.5693161139456007 0.0004949941970051213 -3.0032240932623467e-09
- joint panda_joint3: origin xyz=-4.831237243079438e-05 -0.3160196186961809 8.223830388911502e-05 rpy=1.5701368639143456 0.00021547124952556483 0.00046325645207522415 -> xyz=0.0001883126585843947 -0.31618494823706667 0.00010709261667410667 rpy=1.5700373659353777 0.0004013185711010858 0.0004354649571989922
- joint panda_joint4: origin xyz=0.08218622382442696 0.00012463089813243814 1.9815805120017282e-05 rpy=1.5699691608784458 0.003392401284735163 -0.00022561343078897857 -> xyz=0.08212347014285691 0.0001041932521695015 0.0001851027004233634 rpy=1.5700674172923184 0.0035073747899107355 -0.0004095758957656705
- joint panda_joint5: origin xyz=-0.08161671980459631 0.38418467132228995 -0.0001250123513799326 rpy=-1.5712115657202819 0.0016558929683474796 -0.0030382657944411353 -> xyz=-0.08167007889820048 0.3844213904249064 -0.00010401413491507936 rpy=-1.5712109650464197 0.0014578939249388773 -0.0031542458976239977
- joint panda_joint6: origin xyz=6.629314849055931e-05 0.00045553055999363366 0.00018813569080110683 rpy=1.5680134729931703 8.562990901120595e-05 0.0016569948945247314 -> xyz=-2.547431428789668e-05 0.0004956043554453654 0.00042433833035474894 rpy=1.5685387621185412 7.148845221729656e-05 0.0014592276236294337
- joint panda_joint7: origin xyz=0.08768107566644284 -1.2646922078415426e-05 -0.0004545969030486451 rpy=1.5708928447112276 -1.1846509241174548e-07 -7.997671792020968e-05 -> xyz=0.08776795479481962 -2.0058093454871937e-06 -0.0004945624339437032 rpy=1.5708614097535796 -3.501837319540556e-08 -6.802005614275554e-05
