Commit message: loaded the urdf files in the dual_panda_urdf.xacro. The nice thing is that also the tf are going to be calibrated now. In order to avoid conflict in the joint name definition, I had to modify the single urdf files. This implies that I need to write a script that comverts that automatically or I need to find a smarter to difine the urdf, for example by using a xacro format.

File: description/dual_panda.urdf.xacro (robot description, xacro)
@@ -3,6 +3,4 @@
   <xacro:arg name="arm_id_1" default="panda_right" />
   <xacro:arg name="arm_id_2" default="panda_left" />
-  <xacro:include filename="$(find franka_description)/robots/common/franka_arm.xacro"/>
-  <xacro:include filename="$(find franka_description)/robots/common/franka_hand.xacro"/>
   <!-- box shaped table as base for the 2 Pandas -->
   <link name="base">
@@ -23,4 +21,5 @@
     </collision>
   </link>
+  <!-- <xacro:include filename="$(find franka_description)/robots/common/franka_hand.xacro"/> -->
 <!-- Load the yaml file in franka_bimanual_controllers with relative_position in it -->
   <xacro:property name="relative_position" value="${xacro.load_yaml('$(find franka_bimanual_controllers)/config/relative_position.yaml')}"/>
@@ -37,15 +36,15 @@
   <xacro:property name="left_orientation_p" value="${relative_position['left']['orientation']['p']}"/>
   <xacro:property name="left_orientation_y" value="${relative_position['left']['orientation']['y']}"/>
-  <!-- right arm with gripper -->
-  <xacro:franka_arm arm_id="$(arg arm_id_1)" connected_to="base"  xyz="${right_position_x} ${right_position_y} ${right_position_z}" rpy="${right_orientation_r} ${right_orientation_p} ${right_orientation_y}" safety_distance="0.03" joint_limits="${xacro.load_yaml('$(find franka_description)/robots/panda/joint_limits.yaml')}"/>
-  <xacro:franka_hand arm_id="$(arg arm_id_1)" rpy="0 0 ${-pi/4}" connected_to="$(arg arm_id_1)_link8" safety_distance="0.03"/>
-  <xacro:franka_arm arm_id="$(arg arm_id_2)" connected_to="base"  xyz="${left_position_x} ${left_position_y} ${left_position_z}" rpy="${left_orientation_r} ${left_orientation_p} ${left_orientation_y}" safety_distance="0.03" joint_limits="${xacro.load_yaml('$(find franka_description)/robots/panda/joint_limits.yaml')}"/>
-  <xacro:franka_hand arm_id="$(arg arm_id_2)" rpy="0 0 ${-pi/4}" connected_to="$(arg arm_id_2)_link8" safety_distance="0.03"/>
-    <!-- right arm with gripper -->
-  <!-- <xacro:franka_arm arm_id="$(arg arm_id_1)" connected_to="base"  xyz="0 -0.5 1" rpy="0 0 ${-pi/2}" safety_distance="0.03" joint_limits="${xacro.load_yaml('$(find franka_description)/robots/panda/joint_limits.yaml')}"/>
-  <xacro:franka_hand arm_id="$(arg arm_id_1)" rpy="0 0 ${-pi/4}" connected_to="$(arg arm_id_1)_link8" safety_distance="0.03"/> -->
-  <!-- left arm with gripper -->
-  <!-- <xacro:franka_arm arm_id="$(arg arm_id_2)" connected_to="base"  xyz="0 0.5 1" rpy="0 0 ${pi/2}" safety_distance="0.03" joint_limits="${xacro.load_yaml('$(find franka_description)/robots/panda/joint_limits.yaml')}"/>
-  <xacro:franka_hand arm_id="$(arg arm_id_2)" rpy="0 0 ${-pi/4}" connected_to="$(arg arm_id_2)_link8" safety_distance="0.03"/>
-   -->
+  <joint name="base_to_panda_left_link0" type="fixed">
+    <origin rpy="${left_orientation_r} ${left_orientation_p} ${left_orientation_y}" xyz="${left_position_x} ${left_position_y} ${left_position_z}" />
+    <parent link="base" />
+    <child link="panda_left_link0" />
+  </joint>
+  <joint name="base_to_panda_right_link0" type="fixed">
+    <origin rpy="${right_orientation_r} ${right_orientation_p} ${right_orientation_y}" xyz="${right_position_x} ${right_position_y} ${right_position_z}" />
+    <parent link="base" />
+    <child link="panda_right_link0" />
+  </joint>
+  <xacro:include filename="$(find franka_bimanual_controllers)/urdf/panda_calibrated_right.urdf" />
+  <xacro:include filename="$(find franka_bimanual_controllers)/urdf/panda_calibrated_left.urdf" />
 </robot>

File: urdf/panda_calibrated_left.urdf (robot description, URDF)
Before this commit: robot panda, 14 links, 13 joints
Links:
- removed link ball_link
- removed link panda_hand
- removed link panda_hand_tcp
- removed link panda_leftfinger
- removed link panda_link0
- removed link panda_link1
- removed link panda_link2
- removed link panda_link3
- removed link panda_link4
- removed link panda_link5
- removed link panda_link6
- removed link panda_link7
- removed link panda_link8
- removed link panda_rightfinger
- added link ball_left_link; visual sphere radius=0.005
- added link panda_left_hand; visual mesh filename=package://franka_description/meshes/visual/hand.dae
- added link panda_left_hand_tcp
- added link panda_left_leftfinger; visual mesh filename=package://franka_description/meshes/visual/finger.dae
- added link panda_left_link0; visual mesh filename=package://franka_description/meshes/visual/link0.dae
- added link panda_left_link1; visual mesh filename=package://franka_description/meshes/visual/link1.dae
- added link panda_left_link2; visual mesh filename=package://franka_description/meshes/visual/link2.dae
- added link panda_left_link3; visual mesh filename=package://franka_description/meshes/visual/link3.dae
- added link panda_left_link4; visual mesh filename=package://franka_description/meshes/visual/link4.dae
- added link panda_left_link5; visual mesh filename=package://franka_description/meshes/visual/link5.dae
- added link panda_left_link6; visual mesh filename=package://franka_description/meshes/visual/link6.dae
- added link panda_left_link7; visual mesh filename=package://franka_description/meshes/visual/link7.dae
- added link panda_left_link8
- added link panda_left_rightfinger; visual mesh filename=package://franka_description/meshes/visual/finger.dae
Joints:
- removed joint ball_joint
- removed joint panda_finger_joint1
- removed joint panda_finger_joint2
- removed joint panda_hand_joint
- removed joint panda_hand_tcp_joint
- removed joint panda_joint1
- removed joint panda_joint2
- removed joint panda_joint3
- removed joint panda_joint4
- removed joint panda_joint5
- removed joint panda_joint6
- removed joint panda_joint7
- removed joint panda_joint8
- added joint ball_left_joint: type fixed, parent panda_left_hand_tcp, child ball_left_link, origin xyz=-0.00023049759980861887 0.00044039014121866966 0.031100743489190348 rpy=0.0 0.0 0.0
- added joint panda_left_finger_joint1: type prismatic, parent panda_left_hand, child panda_left_leftfinger, origin xyz=0 0 0.0584 rpy=0 0 0, axis 0 1 0, limit lower=0.0 upper=0.04 effort=100 velocity=0.2
- added joint panda_left_finger_joint2: type prismatic, parent panda_left_hand, child panda_left_rightfinger, origin xyz=0 0 0.0584 rpy=0 0 0, axis 0 -1 0, limit lower=0.0 upper=0.04 effort=100 velocity=0.2, mimic joint=panda_left_finger_joint1
- added joint panda_left_hand_joint: type fixed, parent panda_left_link8, child panda_left_hand, origin xyz=0 0 0 rpy=0 0 -0.7853981633974483
- added joint panda_left_hand_tcp_joint: type fixed, parent panda_left_hand, child panda_left_hand_tcp, origin xyz=0 0 0.1884 rpy=0 0 0
- added joint panda_left_joint1: type revolute, parent panda_left_link0, child panda_left_link1, origin xyz=-1.4596613238343867e-17 -9.055693218673766e-17 0.333 rpy=-1.828892248693048e-17 8.671137250584476e-18 -2.0577862275452234e-17, axis 0 0 1, limit lower=-2.8973 upper=2.8973 effort=87.0 velocity=2.175
- added joint panda_left_joint2: type revolute, parent panda_left_link1, child panda_left_link2, origin xyz=0.00034046892346445374 -0.00027609138626588024 -2.4530901909373608e-17 rpy=-1.5731826118735361 0.0008804625507391334 4.79318753789608e-08, axis 0 0 1, limit lower=-1.7628 upper=1.7628 effort=87.0 velocity=2.175
- added joint panda_left_joint3: type revolute, parent panda_left_link2, child panda_left_link3, origin xyz=0.00011482204889668299 -0.31591360277075664 -0.0002760912953803214 rpy=1.5723422152643884 0.0008208410846264723 0.0008441267498452069, axis 0 0 1, limit lower=-2.8973 upper=2.8973 effort=87.0 velocity=2.175
- added joint panda_left_joint4: type revolute, parent panda_left_link3, child panda_left_link4, origin xyz=0.08225834378378427 -2.2463482153615717e-05 -8.565172079819686e-05 rpy=1.5731556140861436 0.011786197996681824 -0.0008202845766085335, axis 0 0 1, limit lower=-3.0718 upper=-0.0698 effort=87.0 velocity=2.175
- added joint panda_left_joint5: type revolute, parent panda_left_link4, child panda_left_link5, origin xyz=-0.07855928728215028 0.38451520959214897 2.294719504146994e-05 rpy=-1.5706656685042597 0.004904763353391575 -0.010228702256771381, axis 0 0 1, limit lower=-2.8973 upper=2.8973 effort=12.0 velocity=2.61
- added joint panda_left_joint6: type revolute, parent panda_left_link5, child panda_left_link6, origin xyz=0.0006528784687554265 0.00019996069776008653 0.0005556285825519909 rpy=1.5717644448432413 -0.0005146035481431135 0.0049033457862993225, axis 0 0 1, limit lower=-0.0175 upper=3.7525 effort=12.0 velocity=2.61
- added joint panda_left_joint7: type revolute, parent panda_left_link6, child panda_left_link7, origin xyz=0.09024626292728476 -2.4012052499956137e-05 -0.0001973603029375395 rpy=1.5708497729215354 -5.006328509410342e-08 0.0005117785060925037, axis 0 0 1, limit lower=-2.8973 upper=2.8973 effort=12.0 velocity=2.61
- added joint panda_left_joint8: type fixed, parent panda_left_link7, child panda_left_link8, origin xyz=0 0 0.107 rpy=0 0 0

File: urdf/panda_calibrated_right.urdf (robot description, URDF)
Before this commit: robot panda, 14 links, 13 joints
Links:
- removed link ball_link
- removed link panda_hand
- removed link panda_hand_tcp
- removed link panda_leftfinger
- removed link panda_link0
- removed link panda_link1
- removed link panda_link2
- removed link panda_link3
- removed link panda_link4
- removed link panda_link5
- removed link panda_link6
- removed link panda_link7
- removed link panda_link8
- removed link panda_rightfinger
- added link ball_right_link; visual sphere radius=0.005
- added link panda_right_hand; visual mesh filename=package://franka_description/meshes/visual/hand.dae
- added link panda_right_hand_tcp
- added link panda_right_leftfinger; visual mesh filename=package://franka_description/meshes/visual/finger.dae
- added link panda_right_link0; visual mesh filename=package://franka_description/meshes/visual/link0.dae
- added link panda_right_link1; visual mesh filename=package://franka_description/meshes/visual/link1.dae
- added link panda_right_link2; visual mesh filename=package://franka_description/meshes/visual/link2.dae
- added link panda_right_link3; visual mesh filename=package://franka_description/meshes/visual/link3.dae
- added link panda_right_link4; visual mesh filename=package://franka_description/meshes/visual/link4.dae
- added link panda_right_link5; visual mesh filename=package://franka_description/meshes/visual/link5.dae
- added link panda_right_link6; visual mesh filename=package://franka_description/meshes/visual/link6.dae
- added link panda_right_link7; visual mesh filename=package://franka_description/meshes/visual/link7.dae
- added link panda_right_link8
- added link panda_right_rightfinger; visual mesh filename=package://franka_description/meshes/visual/finger.dae
Joints:
- removed joint ball_joint
- removed joint panda_finger_joint1
- removed joint panda_finger_joint2
- removed joint panda_hand_joint
- removed joint panda_hand_tcp_joint
- removed joint panda_joint1
- removed joint panda_joint2
- removed joint panda_joint3
- removed joint panda_joint4
- removed joint panda_joint5
- removed joint panda_joint6
- removed joint panda_joint7
- removed joint panda_joint8
- added joint ball_right_joint: type fixed, parent panda_right_hand_tcp, child ball_right_link, origin xyz=0.0002309827402522288 -0.0004328828032887883 0.03240671849867958 rpy=0.0 0.0 0.0
- added joint panda_right_finger_joint1: type prismatic, parent panda_right_hand, child panda_right_leftfinger, origin xyz=0 0 0.0584 rpy=0 0 0, axis 0 1 0, limit lower=0.0 upper=0.04 effort=100 velocity=0.2
- added joint panda_right_finger_joint2: type prismatic, parent panda_right_hand, child panda_right_rightfinger, origin xyz=0 0 0.0584 rpy=0 0 0, axis 0 -1 0, limit lower=0.0 upper=0.04 effort=100 velocity=0.2, mimic joint=panda_right_finger_joint1
- added joint panda_right_hand_joint: type fixed, parent panda_right_link8, child panda_right_hand, origin xyz=0 0 0 rpy=0 0 -0.7853981633974483
- added joint panda_right_hand_tcp_joint: type fixed, parent panda_right_hand, child panda_right_hand_tcp, origin xyz=0 0 0.1884 rpy=0 0 0
- added joint panda_right_joint1: type revolute, parent panda_right_link0, child panda_right_link1, origin xyz=-6.283931712402919e-18 5.785240799539949e-17 0.333 rpy=2.4213079838489953e-17 -3.589660391516474e-18 -8.469944304901584e-18, axis 0 0 1, limit lower=-2.8973 upper=2.8973 effort=87.0 velocity=2.175
- added joint panda_right_joint2: type revolute, parent panda_right_link1, child panda_right_link2, origin xyz=-0.00010087933252105225 0.0001070930255027192 1.7329529520611466e-17 rpy=-1.5693161139456007 0.0004949941970051213 -3.0032240932623467e-09, axis 0 0 1, limit lower=-1.7628 upper=1.7628 effort=87.0 velocity=2.175
- added joint panda_right_joint3: type revolute, parent panda_right_link2, child panda_right_link3, origin xyz=0.0001883126585843947 -0.31618494823706667 0.00010709261667410667 rpy=1.5700373659353777 0.0004013185711010858 0.0004354649571989922, axis 0 0 1, limit lower=-2.8973 upper=2.8973 effort=87.0 velocity=2.175
- added joint panda_right_joint4: type revolute, parent panda_right_link3, child panda_right_link4, origin xyz=0.08212347014285691 0.0001041932521695015 0.0001851027004233634 rpy=1.5700674172923184 0.0035073747899107355 -0.0004095758957656705, axis 0 0 1, limit lower=-3.0718 upper=-0.0698 effort=87.0 velocity=2.175
- added joint panda_right_joint5: type revolute, parent panda_right_link4, child panda_right_link5, origin xyz=-0.08167007889820048 0.3844213904249064 -0.00010401413491507936 rpy=-1.5712109650464197 0.0014578939249388773 -0.0031542458976239977, axis 0 0 1, limit lower=-2.8973 upper=2.8973 effort=12.0 velocity=2.61
- added joint panda_right_joint6: type revolute, parent panda_right_link5, child panda_right_link6, origin xyz=-2.547431428789668e-05 0.0004956043554453654 0.00042433833035474894 rpy=1.5685387621185412 7.148845221729656e-05 0.0014592276236294337, axis 0 0 1, limit lower=-0.0175 upper=3.7525 effort=12.0 velocity=2.61
- added joint panda_right_joint7: type revolute, parent panda_right_link6, child panda_right_link7, origin xyz=0.08776795479481962 -2.0058093454871937e-06 -0.0004945624339437032 rpy=1.5708614097535796 -3.501837319540556e-08 -6.802005614275554e-05, axis 0 0 1, limit lower=-2.8973 upper=2.8973 effort=12.0 velocity=2.61
- added joint panda_right_joint8: type fixed, parent panda_right_link7, child panda_right_link8, origin xyz=0 0 0.107 rpy=0 0 0
